File: board/SD_Swap/SD_Swap.kicad_sch (KiCad schematic)
At the start: 46 parts, among them J1 USB_C, Q1 Q_Dual_PNP_PNP_E1B1C2E2B2C1, U1 74LVC2G14, U2 RTS5306E, U3 PCB_SD, U4 93AAxxAT, U5 TS3A27518ERTW, U6 SD_SOCKET, U7 AP2127N-3.3, Y1 12MHz

Commit message: add board mostly done
Connections:
- net at U5.1 (COM1): now also U6.8 (DAT1); no longer U6.5 (CLK)
- net at U5.10 (NO2): now also U2.19 (SD_D0); no longer U2.21 (SD_CMD)
- net at U5.12 (NO3): now also U2.20 (SD_CLK); no longer U2.19 (SD_D0)
- net at U5.13 (NO6): now also U2.21 (SD_CMD); no longer U2.22 (SD_D3)
- net at U5.14 (NO4): now also U2.22 (SD_D3); no longer U2.18 (SD_D1)
- net at U5.18 (NC4): now also U3.2 (DAT3); no longer U3.8 (DAT1)
- net at U5.19 (NC6): now also U3.3 (CMD); no longer U3.2 (DAT3)
- net at U5.20 (NC3): now also U3.5 (CLK); no longer U3.7 (DAT0)
- net at U5.22 (NC2): now also U3.7 (DAT0); no longer U3.3 (CMD)
- net at U5.23 (NC1): now also U3.8 (DAT1); no longer U3.5 (CLK)
- net at U5.3 (COM2): now also U6.7 (DAT0); no longer U6.3 (CMD)
- net at U5.4 (COM3): now also U6.5 (CLK); no longer U6.7 (DAT0)
- net at U5.6 (COM4): now also U6.2 (DAT3); no longer U6.8 (DAT1)
- net at U5.8 (NO1): now also U2.18 (SD_D1); no longer U2.20 (SD_CLK)
- net at U5.9 (COM6): now also U6.3 (CMD); no longer U6.2 (DAT3)
Changed lines of the file:
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@@
   (symbol (lib_id "Analog_Switch:TS3A27518ERTW") (at 203.962 51.816 0) (mirror y) (unit 1)
     (in_bom yes) (on_board yes)
-    (property "Reference" "U5" (id 0) (at 188.722 33.02 0)
+    (property "Reference" "U5" (id 0) (at 219.202 33.02 0)
       (effects (font (size 1.27 1.27)) (justify right))
     )

Commit message: add sdcard holder
Parts:
- C1: footprint Capacitor_SMD:C_0603_1608Metric -> SD_Swap:105162-0001
- U6: footprint (none) -> SD_Swap:105162-0001
Connections:
- net GND: now also U6.10 (SHIELD), U6.11 (SHIELD), U6.12 (SHIELD), U6.13 (SHIELD), U6.14 (SHIELD), U6.15 (SHIELD)
Changed lines of the file:
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@@
       (effects (font (size 1.27 1.27)) (justify left))
     )
-    (property "Footprint" "Capacitor_SMD:C_0603_1608Metric" (id 2) (at 130.556 144.018 0)
+    (property "Footprint" "SD_Swap:105162-0001" (id 2) (at 130.556 144.018 0)
       (effects (font (size 1.27 1.27)) hide)
     )
@@
       (effects (font (size 1.27 1.27)) (justify left))
     )
-    (property "Footprint" "" (id 2) (at 240.792 27.051 0)
+    (property "Footprint" "SD_Swap:105162-0001" (id 2) (at 240.792 27.051 0)
       (effects (font (size 1.27 1.27)) hide)
     )
@@
     )
     (pin "1")
+    (pin "10")
+    (pin "11")
+    (pin "12")
+    (pin "13")
+    (pin "14")
+    (pin "15")
     (pin "2")
     (pin "3")
@@
     )
     (path "/09a8b05e-56e6-46dc-90be-1c6b062da039"
-      (reference "C1") (unit 1) (value "~20p") (footprint "Capacitor_SMD:C_0603_1608Metric")
+      (reference "C1") (unit 1) (value "~20p") (footprint "SD_Swap:105162-0001")
     )
     (path "/882eddee-9bf3-4fbf-87b3-0ccbb64aa848"
@@
     )
     (path "/be70e1ce-920b-4f66-b03b-638f9009ed3e"
-      (reference "U6") (unit 1) (value "SD_SOCKET") (footprint "")
+      (reference "U6") (unit 1) (value "SD_SOCKET") (footprint "SD_Swap:105162-0001")
     )
     (path "/9fc772fc-7a92-45cc-a80f-b1ab89f05f6f"
